File: KiCad/MacroPad.sch (KiCad schematic (older format))
At the start: 41 parts, among them J1 USB_OTG, SW1 SW_Push, SW10 SW_Push, SW11 SW_Push, SW12 SW_Push, SW2 SW_Push, SW3 SW_Push, SW4 SW_Push, SW5 SW_Push, SW50 RESET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

Commit message: Keyboard schematic with associated parts
Parts:
- removed F1: 100mA, symbol Device:Polyfuse_Small
- C1, C2: footprint (none) -> Capacitor_THT:C_Disc_D3.0mm_W1.6mm_P2.50mm
- C3: footprint (none) -> Capacitor_THT:CP_Radial_D4.0mm_P1.50mm
- C4, C5: footprint (none) -> Capacitor_THT:C_Disc_D4.3mm_W1.9mm_P5.00mm
- D1, D10, D11, D12, D2, D3, D4, D49, D5, D50, D6, D7, D8, D9: footprint (none) -> Diode_THT:D_DO-35_SOD27_P5.08mm_Vertical_KathodeUp
- J1, R1: footprint (none) -> Connector_USB:USB_Mini-B_Lumberg_2486_01_Horizontal
- R2, R3, R4: footprint (none) -> Resistor_THT:R_Axial_DIN0204_L3.6mm_D1.6mm_P5.08mm_Horizontal
- SW1, SW10, SW11, SW12, SW2, SW3, SW4, SW5, SW6, SW7, SW8, SW9: footprint (none) -> SMKJP:SW_Cherry_MX1A_1.00u_PCB
- SW50, SW51: footprint (none) -> Button_Switch_THT:SW_PUSH_6mm
- Y1: footprint (none) -> Crystal:Crystal_HC49-4H_Vertical
- gave numbers to parts that had none: 1
Connections:
- net +5V: now also J1.1 (VBUS)
- no-connect marks 3 -> 13

Commit message: Arrange components for size analysis with accurate mx switches
Parts:
- R1: footprint Connector_USB:USB_Mini-B_Lumberg_2486_01_Horizontal -> Resistor_THT:R_Axial_DIN0204_L3.6mm_D1.6mm_P5.08mm_Horizontal
Changed lines of the file:
@@
 F 0 "R1" V 2400 2900 50  0000 L CNN
 F 1 "1.5k" V 2600 2950 50  0000 C CNN
-F 2 "Connector_USB:USB_Mini-B_Lumberg_2486_01_Horizontal" H 2500 2950 50  0001 C CNN
+F 2 "Resistor_THT:R_Axial_DIN0204_L3.6mm_D1.6mm_P5.08mm_Horizontal" H 2500 2950 50  0001 C CNN
 F 3 "~" H 2500 2950 50  0001 C CNN
 	1    2500 2950
