File: Eagle_2/MacroPad.sch (EAGLE design)
At the start: 42 parts, among them SW00 SWITCH-SMD-EVQP-P2602W, SW01 KEYSWITCH-PLAIN-MX-1U, SW02 KEYSWITCH-PLAIN-MX-1U, SW03 KEYSWITCH-PLAIN-MX-1U, SW04 KEYSWITCH-PLAIN-MX-1U, SW05 KEYSWITCH-PLAIN-MX-1U, SW06 KEYSWITCH-PLAIN-MX-1U, SW07 KEYSWITCH-PLAIN-MX-1U, SW08 KEYSWITCH-PLAIN-MX-1U, SW09 KEYSWITCH-PLAIN-MX-1U, SW10 KEYSWITCH-PLAIN-MX-1U, SW11 KEYSWITCH-PLAIN-MX-1U, SW12 KEYSWITCH-PLAIN-MX-1U

Commit message: Add Bill of Materials and README
Parts:
- C1, C2: MPN (none) -> 04025A220JAT2A; OC_NEWARK (none) -> 96M1143
- C3, C4, C5, C6, C7, C8, C9, D1, D10, D11, D12, D2, D3, D4, D5, D6, D7, D8, D9, F1, R1, R2, R3, R4, SW00, SW01, SW02, SW03, SW04, SW05, SW06, SW07, SW08, SW09, SW10, SW11, SW12, U$1, USB1, Y1: OC_NEWARK (none) -> unknown
